Commit message: Bug in ros2 control

File: src/magbot_gazebo/description/backup/dingo.urdf (robot description, URDF)
Before this commit: robot dingo, 17 links, 16 joints
Links:
- added link world_link
- link FL_link1: mass 0.30000000 -> 0.2
- link FL_link2: mass 0.10000000 -> 0.05
- link FL_link3: mass 0.10000000 -> 0.05
- link FL_link4: mass 0.02000000 -> 0.01
- link FR_link1: mass 0.30000000 -> 0.2
- link FR_link2: mass 0.10000000 -> 0.05
- link FR_link3: mass 0.10000000 -> 0.05
- link FR_link4: mass 0.02000000 -> 0.01
- link RL_link1: mass 0.30000000 -> 0.2
- link RL_link2: mass 0.10000000 -> 0.05
- link RL_link3: mass 0.10000000 -> 0.05
- link RL_link4: mass 0.02000000 -> 0.01
- link RR_link1: mass 0.30000000 -> 0.2
- link RR_link2: mass 0.10000000 -> 0.05
- link RR_link3: mass 0.10000000 -> 0.05
- link RR_link4: mass 0.02000000 -> 0.01
- link base_link: mass 0.81776 -> 2.2
Joints:
- added joint world_to_base: type fixed, parent world_link, child base_link

File: src/magbot_gazebo/description/urdf/dingo.urdf.xacro (robot description, xacro)
@@ -1,17 +1,25 @@
 <robot name="dingo" xmlns:xacro="http://www.ros.org/wiki/xacro">
+  <!-- Maximum torque -->
   <xacro:include filename="$(find magbot_gazebo)/description/urdf/dingo_ros2_control.xacro" />
   <!-- Maximum torque -->
   <xacro:property name="effort_limit" value="10" />
-  <!-- The root link can't have inertia so did this -->
-  <!-- <link name="root_dummy_link" />
-  <joint name="root_joint" type="fixed">
-    <parent link="root_dummy_link"/>
-    <child link="base_link"/>
-  </joint> -->
-  <!-- The root link can't have inertia so did this -->
   <!-- base_link -->
   <link
     name="base_link">
     <!-- <inertial>
+      <origin xyz="0.0 0.0 0.0"/>
+      <mass value="2.50000000"/>
+      <inertia ixx="0.00664756" ixy="0.00002187" ixz="0.00015428" iyy="0.02996945" iyz="-0.00000064"
+    izz="0.03274274"/>
+    </inertial>-->
+    <!--
+    <inertial>
+      <origin xyz="0.0 0.00126483 -0.00622132"/>
+      <mass value="2.5000000"/>
+      <inertia ixx="0.00664756" ixy="0.00002187" ixz="0.00015428" iyy="0.02996945" iyz="-0.00000064"
+    izz="0.03274274"/>
+    </inertial>
+    -->
+    <inertial>
       <origin
         xyz="0 0 0"
@@ -26,10 +34,13 @@
         iyz="3.2027E-08"
         izz="0.00063853" />
-    </inertial> -->
+    </inertial>
+    <!--
     <inertial>
       <origin xyz="-0.02679290 -0.00012097 0.00457177"/>
       <mass value="5.0000000"/>
-      <inertia ixx="0.00732760" ixy="-0.00000000" ixz="0.00021940" iyy="0.02995798" iyz="-0.00000002" izz="0.03298004"/>
-    </inertial>
+      <inertia ixx="0.00732760" ixy="-0.00000000" ixz="0.00021940" iyy="0.02995798" iyz="-0.00000002"
+    izz="0.03298004"/>
+    </inertial>
+    -->
     <visual>
       <origin
@@ -40,6 +51,8 @@
           filename="package://magbot_gazebo/description/meshes/base_link.dae" />
       </geometry>
-      <material name="">
-        <color rgba="0.15294 0.78431 0.96078 1" />
+      <material
+        name="">
+        <color
+          rgba="0.79216 0.81961 0.93333 1" />
       </material>
     </visual>
@@ -58,7 +71,8 @@
     name="FL_link1">
     <inertial>
-      <origin xyz="0 0 0"/>
-      <mass value="0.30000000"/>
-      <inertia ixx="0.00019300" ixy="0.00000000" ixz="0.00000000" iyy="0.00014890" iyz="0.00000000" izz="0.00012410"/>
+      <origin xyz="0 0 0" />
+      <mass value="0.30000000" />
+      <inertia ixx="0.00019300" ixy="0.00000000" ixz="0.00000000" iyy="0.00014890" iyz="0.00000000"
+        izz="0.00012410" />
     </inertial>
     <visual>
@@ -70,6 +84,8 @@
           filename="package://magbot_gazebo/description/meshes/FL_link1.dae" />
       </geometry>
-      <material name="">
-        <color rgba="0.15294 0.78431 0.96078 1" />
+      <material
+        name="">
+        <color
+          rgba="0.79216 0.81961 0.93333 1" />
       </material>
     </visual>
@@ -88,7 +104,8 @@
     name="FL_link2">
     <inertial>
-      <origin xyz="0 0 0"/>
-      <mass value="0.10000000"/>
-      <inertia ixx="0.00000700" ixy="0.00000000" ixz="0.00000444" iyy="0.00017260" iyz="0.00000000" izz="0.00017568"/>
+      <origin xyz="0 0 0" />
+      <mass value="0.10000000" />
+      <inertia ixx="0.00000700" ixy="0.00000000" ixz="0.00000444" iyy="0.00017260" iyz="0.00000000"
+        izz="0.00017568" />
     </inertial>
     <visual>
@@ -100,6 +117,8 @@
           filename="package://magbot_gazebo/description/meshes/L_link2.dae" />
       </geometry>
-      <material name="">
-        <color rgba="0.15294 0.78431 0.96078 1" />
+      <material
+        name="">
+        <color
+          rgba="0.79216 0.81961 0.93333 1" />
       </material>
     </visual>
@@ -118,7 +137,8 @@
     name="FL_link3">
     <inertial>
-      <origin xyz="0 0 0"/>
-      <mass value="0.10000000"/>
-      <inertia ixx="0.00000936" ixy="-0.00001360" ixz="-0.00000319" iyy="0.00019747" iyz="-0.00000027" izz="0.00019702"/>
+      <origin xyz="0 0 0" />
+      <mass value="0.10000000" />
+      <inertia ixx="0.00000936" ixy="-0.00001360" ixz="-0.00000319" iyy="0.00019747"
+        iyz="-0.00000027" izz="0.00019702" />
     </inertial>
     <visual>
@@ -130,6 +150,8 @@
           filename="package://magbot_gazebo/description/meshes/L_link3.dae" />
       </geometry>
-      <material name="">
-        <color rgba="0.15294 0.78431 0.96078 1" />
+      <material
+        name="">
+        <color
+          rgba="0.79216 0.81961 0.93333 1" />
       </material>
     </visual>
@@ -148,7 +170,8 @@
     name="FL_link4">
     <inertial>
-      <origin xyz="0 0 0"/>
-      <mass value="0.02000000"/>
-      <inertia ixx="0.00000060" ixy="-0.00000013" ixz="0.00000000" iyy="0.00000058" iyz="0.00000000" izz="0.00000045"/>
+      <origin xyz="0 0 0" />
+      <mass value="0.02000000" />
+      <inertia ixx="0.00000060" ixy="-0.00000013" ixz="0.00000000" iyy="0.00000058" iyz="0.00000000"
+        izz="0.00000045" />
     </inertial>
     <visual>
@@ -160,6 +183,8 @@
           filename="package://magbot_gazebo/description/meshes/link4.dae" />
       </geometry>
-      <material name="">
-        <color rgba="0.15294 0.78431 0.96078 1" />
+      <material
+        name="">
+        <color
+          rgba="0.79216 0.81961 0.93333 1" />
       </material>
     </visual>
@@ -178,7 +203,8 @@
     name="FR_link1">
     <inertial>
-      <origin xyz="0 0 0"/>
-      <mass value="0.30000000"/>
-      <inertia ixx="0.00019300" ixy="0.00000000" ixz="0.00000000" iyy="0.00014890" iyz="0.00000000" izz="0.00012410"/>
+      <origin xyz="0 0 0" />
+      <mass value="0.30000000" />
+      <inertia ixx="0.00019300" ixy="0.00000000" ixz="0.00000000" iyy="0.00014890" iyz="0.00000000"
+        izz="0.00012410" />
     </inertial>
     <visual>
@@ -190,6 +216,8 @@
           filename="package://magbot_gazebo/description/meshes/FR_link1.dae" />
       </geometry>
-      <material name="">
-        <color rgba="0.15294 0.78431 0.96078 1" />
+      <material
+        name="">
+        <color
+          rgba="0.79216 0.81961 0.93333 1" />
       </material>
     </visual>
@@ -208,7 +236,8 @@
     name="FR_link2">
     <inertial>
-      <origin xyz="0 0 0"/>
-      <mass value="0.10000000"/>
-      <inertia ixx="0.00000700" ixy="0.00000000" ixz="0.00000444" iyy="0.00017260" iyz="0.00000000" izz="0.00017568"/>
+      <origin xyz="0 0 0" />
+      <mass value="0.10000000" />
+      <inertia ixx="0.00000700" ixy="0.00000000" ixz="0.00000444" iyy="0.00017260" iyz="0.00000000"
+        izz="0.00017568" />
     </inertial>
     <visual>
@@ -220,6 +249,8 @@
           filename="package://magbot_gazebo/description/meshes/R_link2.dae" />
       </geometry>
-      <material name="">
-        <color rgba="0.15294 0.78431 0.96078 1" />
+      <material
+        name="">
+        <color
+          rgba="0.79216 0.81961 0.93333 1" />
       </material>
     </visual>
@@ -238,7 +269,8 @@
     name="FR_link3">
     <inertial>
-      <origin xyz="0 0 0"/>
-      <mass value="0.10000000"/>
-      <inertia ixx="0.00000936" ixy="-0.00001360" ixz="-0.00000319" iyy="0.00019747" iyz="-0.00000027" izz="0.00019702"/>
+      <origin xyz="0 0 0" />
+      <mass value="0.10000000" />
+      <inertia ixx="0.00000936" ixy="-0.00001360" ixz="-0.00000319" iyy="0.00019747"
+        iyz="-0.00000027" izz="0.00019702" />
     </inertial>
     <visual>
@@ -250,6 +282,8 @@
           filename="package://magbot_gazebo/description/meshes/R_link3.dae" />
       </geometry>
-      <material name="">
-        <color rgba="0.15294 0.78431 0.96078 1" />
+      <material
+        name="">
+        <color
+          rgba="0.79216 0.81961 0.93333 1" />
       </material>
     </visual>
@@ -268,7 +302,8 @@
     name="FR_link4">
     <inertial>
-      <origin xyz="0 0 0"/>
-      <mass value="0.02000000"/>
-      <inertia ixx="0.00000060" ixy="-0.00000013" ixz="0.00000000" iyy="0.00000058" iyz="0.00000000" izz="0.00000045"/>
+      <origin xyz="0 0 0" />
+      <mass value="0.02000000" />
+      <inertia ixx="0.00000060" ixy="-0.00000013" ixz="0.00000000" iyy="0.00000058" iyz="0.00000000"
+        izz="0.00000045" />
     </inertial>
     <visual>
@@ -280,6 +315,8 @@
           filename="package://magbot_gazebo/description/meshes/link4.dae" />
       </geometry>
-      <material name="">
-        <color rgba="0.15294 0.78431 0.96078 1" />
+      <material
+        name="">
+        <color
+          rgba="0.79216 0.81961 0.93333 1" />
       </material>
     </visual>
@@ -298,7 +335,8 @@
     name="RL_link1">
     <inertial>
-      <origin xyz="0 0 0"/>
-      <mass value="0.30000000"/>
-      <inertia ixx="0.00019300" ixy="0.00000000" ixz="0.00000000" iyy="0.00014890" iyz="0.00000000" izz="0.00012410"/>
+      <origin xyz="0 0 0" />
+      <mass value="0.30000000" />
+      <inertia ixx="0.00019300" ixy="0.00000000" ixz="0.00000000" iyy="0.00014890" iyz="0.00000000"
+        izz="0.00012410" />
     </inertial>
     <visual>
@@ -310,6 +348,8 @@
           filename="package://magbot_gazebo/description/meshes/RL_link1.dae" />
       </geometry>
-      <material name="">
-        <color rgba="0.15294 0.78431 0.96078 1" />
+      <material
+        name="">
+        <color
+          rgba="0.79216 0.81961 0.93333 1" />
       </material>
     </visual>
@@ -328,7 +368,8 @@
     name="RL_link2">
     <inertial>
-      <origin xyz="0 0 0"/>
-      <mass value="0.10000000"/>
-      <inertia ixx="0.00000700" ixy="0.00000000" ixz="0.00000444" iyy="0.00017260" iyz="0.00000000" izz="0.00017568"/>
+      <origin xyz="0 0 0" />
+      <mass value="0.10000000" />
+      <inertia ixx="0.00000700" ixy="0.00000000" ixz="0.00000444" iyy="0.00017260" iyz="0.00000000"
+        izz="0.00017568" />
     </inertial>
     <visual>
@@ -340,6 +381,8 @@
           filename="package://magbot_gazebo/description/meshes/L_link2.dae" />
       </geometry>
-      <material name="">
-        <color rgba="0.15294 0.78431 0.96078 1" />
+      <material
+        name="">
+        <color
+          rgba="0.79216 0.81961 0.93333 1" />
       </material>
     </visual>
@@ -358,7 +401,8 @@
     name="RL_link3">
     <inertial>
-      <origin xyz="0 0 0"/>
-      <mass value="0.10000000"/>
-      <inertia ixx="0.00000936" ixy="-0.00001360" ixz="-0.00000319" iyy="0.00019747" iyz="-0.00000027" izz="0.00019702"/>
+      <origin xyz="0 0 0" />
+      <mass value="0.10000000" />
+      <inertia ixx="0.00000936" ixy="-0.00001360" ixz="-0.00000319" iyy="0.00019747"
+        iyz="-0.00000027" izz="0.00019702" />
     </inertial>
     <visual>
@@ -370,6 +414,8 @@
           filename="package://magbot_gazebo/description/meshes/L_link3.dae" />
       </geometry>
-      <material name="">
-        <color rgba="0.15294 0.78431 0.96078 1" />
+      <material
+        name="">
+        <color
+          rgba="0.79216 0.81961 0.93333 1" />
       </material>
     </visual>
@@ -388,7 +434,8 @@
     name="RL_link4">
     <inertial>
-      <origin xyz="0 0 0"/>
-      <mass value="0.02000000"/>
-      <inertia ixx="0.00000060" ixy="-0.00000013" ixz="0.00000000" iyy="0.00000058" iyz="0.00000000" izz="0.00000045"/>
+      <origin xyz="0 0 0" />
+      <mass value="0.02000000" />
+      <inertia ixx="0.00000060" ixy="-0.00000013" ixz="0.00000000" iyy="0.00000058" iyz="0.00000000"
+        izz="0.00000045" />
     </inertial>
     <visual>
@@ -400,6 +447,8 @@
           filename="package://magbot_gazebo/description/meshes/link4.dae" />
       </geometry>
-      <material name="">
-        <color rgba="0.15294 0.78431 0.96078 1" />
+      <material
+        name="">
+        <color
+          rgba="0.79216 0.81961 0.93333 1" />
       </material>
     </visual>
@@ -418,7 +467,8 @@
     name="RR_link1">
     <inertial>
-      <origin xyz="0 0 0"/>
-      <mass value="0.30000000"/>
-      <inertia ixx="0.00019300" ixy="0.00000000" ixz="0.00000000" iyy="0.00014890" iyz="0.00000000" izz="0.00012410"/>
+      <origin xyz="0 0 0" />
+      <mass value="0.30000000" />
+      <inertia ixx="0.00019300" ixy="0.00000000" ixz="0.00000000" iyy="0.00014890" iyz="0.00000000"
+        izz="0.00012410" />
     </inertial>
     <visual>
@@ -430,6 +480,8 @@
           filename="package://magbot_gazebo/description/meshes/RR_link1.dae" />
       </geometry>
-      <material name="">
-        <color rgba="0.15294 0.78431 0.96078 1" />
+      <material
+        name="">
+        <color
+          rgba="0.79216 0.81961 0.93333 1" />
       </material>
     </visual>
@@ -448,7 +500,8 @@
     name="RR_link2">
     <inertial>
-      <origin xyz="0 0 0"/>
-      <mass value="0.10000000"/>
-      <inertia ixx="0.00000700" ixy="0.00000000" ixz="0.00000444" iyy="0.00017260" iyz="0.00000000" izz="0.00017568"/>
+      <origin xyz="0 0 0" />
+      <mass value="0.10000000" />
+      <inertia ixx="0.00000700" ixy="0.00000000" ixz="0.00000444" iyy="0.00017260" iyz="0.00000000"
+        izz="0.00017568" />
     </inertial>
     <visual>
@@ -460,6 +513,8 @@
           filename="package://magbot_gazebo/description/meshes/R_link2.dae" />
       </geometry>
-      <material name="">
-        <color rgba="0.15294 0.78431 0.96078 1" />
+      <material
+        name="">
+        <color
+          rgba="0.79216 0.81961 0.93333 1" />
       </material>
     </visual>
@@ -478,7 +533,8 @@
     name="RR_link3">
     <inertial>
-      <origin xyz="0 0 0"/>
-      <mass value="0.10000000"/>
-      <inertia ixx="0.00000936" ixy="-0.00001360" ixz="-0.00000319" iyy="0.00019747" iyz="-0.00000027" izz="0.00019702"/>
+      <origin xyz="0 0 0" />
+      <mass value="0.10000000" />
+      <inertia ixx="0.00000936" ixy="-0.00001360" ixz="-0.00000319" iyy="0.00019747"
+        iyz="-0.00000027" izz="0.00019702" />
     </inertial>
     <visual>
@@ -490,6 +546,8 @@
           filename="package://magbot_gazebo/description/meshes/R_link3.dae" />
       </geometry>
-      <material name="">
-        <color rgba="0.15294 0.78431 0.96078 1" />
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