Commit message: WIP: Dockerfile + ros2_control loaded

File: src/magbot_gazebo/description/urdf/dingo.urdf.xacro (robot description, xacro)
@@ -819,4 +819,7 @@
     <plugin name="gazebo_ros2_control" filename="libgazebo_ros2_control.so">
       <parameters>$(find magbot_gazebo)/config/dingo_controllers.yaml</parameters>
+       <!-- <ros>
+       <namespace>/dingo_controller</namespace>
+     </ros> -->
     </plugin>
   </gazebo>

File: src/magbot_gazebo/description/urdf/dingo_ros2_control.xacro (robot description, xacro)
@@ -6,9 +6,26 @@
         <plugin>gazebo_ros2_control/GazeboSystem</plugin>
       </hardware>
+      <!-- FL Joint Group -->
+      <joint name="FL_theta1">
+        <command_interface name="position"/>
+        <state_interface name="position"/>
+        <state_interface name="velocity"/>
+        <state_interface name="effort"/>
+      </joint>
+      <joint name="FL_theta2">
+        <command_interface name="position"/>
+        <state_interface name="position"/>
+        <state_interface name="velocity"/>
+        <state_interface name="effort"/>
+      </joint>
+      <joint name="FL_theta3">
+        <command_interface name="position"/>
+        <state_interface name="position"/>
+        <state_interface name="velocity"/>
+        <state_interface name="effort"/>
+      </joint>
+      <!-- FR Joint Group -->
       <joint name="FR_theta1">
-        <command_interface name="effort">
-          <param name="min">-${effort_limit}</param>
-          <param name="max">${effort_limit}</param>
-        </command_interface>
+        <command_interface name="position"/>
         <state_interface name="position"/>
         <state_interface name="velocity"/>
@@ -16,8 +33,5 @@
       </joint>
       <joint name="FR_theta2">
-        <command_interface name="effort">
-          <param name="min">-${effort_limit}</param>
-          <param name="max">${effort_limit}</param>
-        </command_interface>
+        <command_interface name="position"/>
         <state_interface name="position"/>
         <state_interface name="velocity"/>
@@ -25,44 +39,12 @@
       </joint>
       <joint name="FR_theta3">
-        <command_interface name="effort">
-          <param name="min">-${effort_limit}</param>
-          <param name="max">${effort_limit}</param>
-        </command_interface>
+        <command_interface name="position"/>
         <state_interface name="position"/>
         <state_interface name="velocity"/>
         <state_interface name="effort"/>
       </joint>
-      <joint name="FL_theta1">
-        <command_interface name="effort">
-          <param name="min">-${effort_limit}</param>
-          <param name="max">${effort_limit}</param>
-        </command_interface>
-        <state_interface name="position"/>
-        <state_interface name="velocity"/>
-        <state_interface name="effort"/>
-      </joint>
-      <joint name="FL_theta2">
-        <command_interface name="effort">
-          <param name="min">-${effort_limit}</param>
-          <param name="max">${effort_limit}</param>
-        </command_interface>
-        <state_interface name="position"/>
-        <state_interface name="velocity"/>
-        <state_interface name="effort"/>
-      </joint>
-      <joint name="FL_theta3">
-        <command_interface name="effort">
-          <param name="min">-${effort_limit}</param>
-          <param name="max">${effort_limit}</param>
-        </command_interface>
-        <state_interface name="position"/>
-        <state_interface name="velocity"/>
-        <state_interface name="effort"/>
-      </joint>
+      <!-- RR Joint Group -->
       <joint name="RR_theta1">
-        <command_interface name="effort">
-          <param name="min">-${effort_limit}</param>
-          <param name="max">${effort_limit}</param>
-        </command_interface>
+        <command_interface name="position"/>
         <state_interface name="position"/>
         <state_interface name="velocity"/>
@@ -70,8 +52,5 @@
       </joint>
       <joint name="RR_theta2">
-        <command_interface name="effort">
-          <param name="min">-${effort_limit}</param>
-          <param name="max">${effort_limit}</param>
-        </command_interface>
+        <command_interface name="position"/>
         <state_interface name="position"/>
         <state_interface name="velocity"/>
@@ -79,17 +58,12 @@
       </joint>
       <joint name="RR_theta3">
-        <command_interface name="effort">
-          <param name="min">-${effort_limit}</param>
-          <param name="max">${effort_limit}</param>
-        </command_interface>
+        <command_interface name="position"/>
         <state_interface name="position"/>
         <state_interface name="velocity"/>
         <state_interface name="effort"/>
       </joint>
+      <!-- RL Joint Group -->
       <joint name="RL_theta1">
-        <command_interface name="effort">
-          <param name="min">-${effort_limit}</param>
-          <param name="max">${effort_limit}</param>
-        </command_interface>
+        <command_interface name="position"/>
         <state_interface name="position"/>
         <state_interface name="velocity"/>
@@ -97,8 +71,5 @@
       </joint>
       <joint name="RL_theta2">
-        <command_interface name="effort">
-          <param name="min">-${effort_limit}</param>
-          <param name="max">${effort_limit}</param>
-        </command_interface>
+        <command_interface name="position"/>
         <state_interface name="position"/>
         <state_interface name="velocity"/>
@@ -106,8 +77,5 @@
       </joint>
       <joint name="RL_theta3">
-        <command_interface name="effort">
-          <param name="min">-${effort_limit}</param>
-          <param name="max">${effort_limit}</param>
-        </command_interface>
+        <command_interface name="position"/>
         <state_interface name="position"/>
         <state_interface name="velocity"/>
