Commit message: Modified URDF Transmission to newer syntax

File: src/magbot_gazebo/description/urdf/dingo.urdf.xacro (robot description, xacro)
@@ -547,5 +547,6 @@
       effort="${effort_limit}"
       velocity="3" />
-    <joint_properties damping="1000.0" friction="1000.0"/>
+    <!-- <joint_properties damping="1000.0" friction="1000.0"/> -->
+    <dynamics damping="1000.0" friction="1000.0"/>
   </joint>
   <joint
@@ -566,5 +567,6 @@
       effort="${effort_limit}"
       velocity="3" />
-    <joint_properties damping="1000.0" friction="1000.0"/>
+    <!-- <joint_properties damping="1000.0" friction="1000.0"/> -->
+    <dynamics damping="1000.0" friction="1000.0"/>
   </joint>
   <joint
@@ -585,5 +587,6 @@
       effort="${effort_limit}"
       velocity="3" />
-    <joint_properties damping="1000.0" friction="1000.0"/>
+    <!-- <joint_properties damping="1000.0" friction="1000.0"/> -->
+    <dynamics damping="1000.0" friction="1000.0"/>
   </joint>
   <joint
@@ -617,5 +620,6 @@
       effort="${effort_limit}"
       velocity="3" />
-    <joint_properties damping="1000.0" friction="1000.0"/>
+    <!-- <joint_properties damping="1000.0" friction="1000.0"/> -->
+    <dynamics damping="1000.0" friction="1000.0"/>
   </joint>
   <joint
@@ -636,5 +640,6 @@
       effort="${effort_limit}"
       velocity="3" />
-    <joint_properties damping="1000.0" friction="1000.0"/>
+    <!-- <joint_properties damping="1000.0" friction="1000.0"/> -->
+    <dynamics damping="1000.0" friction="1000.0"/>
   </joint>
   <joint
@@ -655,5 +660,6 @@
       effort="${effort_limit}"
       velocity="3" />
-    <joint_properties damping="1000.0" friction="1000.0"/>
+    <!-- <joint_properties damping="1000.0" friction="1000.0"/> -->
+    <dynamics damping="1000.0" friction="1000.0"/>
   </joint>
   <joint
@@ -687,5 +693,6 @@
       effort="${effort_limit}"
       velocity="3" />
-    <joint_properties damping="1000.0" friction="1000.0"/>
+    <!-- <joint_properties damping="1000.0" friction="1000.0"/> -->
+    <dynamics damping="1000.0" friction="1000.0"/>
   </joint>
   <joint
@@ -706,5 +713,6 @@
       effort="${effort_limit}"
       velocity="3" />
-    <joint_properties damping="1000.0" friction="1000.0"/>
+    <!-- <joint_properties damping="1000.0" friction="1000.0"/> -->
+    <dynamics damping="1000.0" friction="1000.0"/>
   </joint>
   <joint
@@ -725,5 +733,6 @@
       effort="${effort_limit}"
       velocity="3" />
-    <joint_properties damping="1000.0" friction="1000.0"/>
+    <!-- <joint_properties damping="1000.0" friction="1000.0"/> -->
+    <dynamics damping="1000.0" friction="1000.0"/>
   </joint>
   <joint
@@ -757,5 +766,6 @@
       effort="${effort_limit}"
       velocity="3" />
-    <joint_properties damping="1000.0" friction="1000.0"/>
+    <!-- <joint_properties damping="1000.0" friction="1000.0"/> -->
+    <dynamics damping="1000.0" friction="1000.0"/>
   </joint>
   <joint
@@ -776,5 +786,6 @@
       effort="${effort_limit}"
       velocity="3" />
-    <joint_properties damping="1000.0" friction="1000.0"/>
+    <!-- <joint_properties damping="1000.0" friction="1000.0"/> -->
+    <dynamics damping="1000.0" friction="1000.0"/>
   </joint>
   <joint
@@ -795,5 +806,6 @@
       effort="${effort_limit}"
       velocity="3" />
-    <joint_properties damping="1000.0" friction="1000.0"/>
+    <!-- <joint_properties damping="1000.0" friction="1000.0"/> -->
+    <dynamics damping="1000.0" friction="1000.0"/>
   </joint>
   <joint
@@ -810,10 +822,4 @@
       xyz="0 0 0" />
   </joint>
-  <!-- ROS control plugin -->
-  <!-- <gazebo>
-    <plugin name="gazebo_ros_control" filename="libgazebo_ros_control.so">
-      <robotNamespace>dingo_controller</robotNamespace>
-    </plugin>
-  </gazebo> -->
   <gazebo>
     <plugin name="gazebo_ros2_control" filename="libgazebo_ros2_control.so">
@@ -824,49 +830,4 @@
     </plugin>
   </gazebo>
-  <!-- IMU sensor -->
-  <!-- <gazebo reference="base_link">
-    <gravity>true</gravity>
-    <sensor name="imu_sensor" type="imu">
-      <always_on>true</always_on>
-      <update_rate>100</update_rate>
-      <visualize>true</visualize>
-      <topic>__default_topic__</topic>
-      <plugin filename="libgazebo_ros_imu_sensor.so" name="imu_plugin">
-        <topicName>notspot_imu/base_link_orientation</topicName>
-        <bodyName>imu_link</bodyName>
-        <updateRateHZ>15.0</updateRateHZ>
-        <gaussianNoise>0.0</gaussianNoise>
-        <xyzOffset>0 0 0</xyzOffset>
-        <rpyOffset>0 0 0</rpyOffset>
-        <frameName>base_link</frameName>
-        <initialOrientationAsReference>false</initialOrientationAsReference>
-      </plugin>
-      <pose>0 0 0 0 0 0</pose>
-    </sensor>
-  </gazebo> -->
-  <!-- Noise might be causing an issue -->
-  <!-- <gazebo reference="base_link">
-    <gravity>true</gravity>
-    <sensor name="imu_sensor" type="imu">
-      <always_on>true</always_on>
-      <update_rate>100</update_rate>
-      <visualize>true</visualize>
-      <topic>__default_topic__</topic>
-      <plugin filename="libgazebo_ros_imu_sensor.so" name="imu_plugin">
-        <ros>
-          <namespace>/dingo</namespace>
-          <remapping>~/out:=imu</remapping>
-        </ros>
-        <topicName>imu</topicName>
-        <bodyName>base_link</bodyName>
-        <updateRateHZ>15.0</updateRateHZ>
-        <gaussianNoise>0.0</gaussianNoise>
-        <xyzOffset>0 0 0</xyzOffset>
-        <rpyOffset>0 0 0</rpyOffset>
-        <frameName>base_link</frameName>
-      </plugin>
-      <pose>0 0 0 0 0 0</pose>
-    </sensor>
-  </gazebo> -->
   <gazebo reference="base_link">
     <gravity>true</gravity>
@@ -907,18 +868,8 @@
     </sensor>
   </gazebo>
-  <!-- Joint state publisher plugin -->
-  <!-- <gazebo>
-    <plugin name="joint_state_publisher" filename="libgazebo_ros_joint_state_publisher.so">
-        <robotNamespace>dingo_gazebo</robotNamespace>
-        <jointName>FR_theta1, FR_theta2, FR_theta3, FL_theta1, FL_theta2,
-                   FL_theta3, RR_theta1, RR_theta2, RR_theta3, RL_theta1,
-                   RL_theta2, RL_theta3</jointName>
-        <updateRate>100</updateRate>
-    </plugin>
-  </gazebo> -->
   <gazebo>
     <plugin name="joint_state_publisher" filename="libgazebo_ros_joint_state_publisher.so">
       <ros>
-        <namespace>/dingo</namespace>
+        <namespace>/dingo_gazebo</namespace>
         <remapping>~/out:=joint_states</remapping>
       </ros>
@@ -939,21 +890,21 @@
   </gazebo>
   <!-- Transmission -->
-  <transmission name="tran1">
+  <!-- <transmission name="tran1">
     <type>transmission_interface/SimpleTransmission</type>
     <joint name="FR_theta1">
-      <hardwareInterface>hardware_interface/JointCommandInterface</hardwareInterface>
+      <hardwareInterface>hardware_interface/PositionJointInterface</hardwareInterface>
     </joint>
     <actuator name="motor1">
-    <hardwareInterface>hardware_interface/JointCommandInterface</hardwareInterface>
-    <mechanicalReduction>5</mechanicalReduction>
-    </actuator>
-  </transmission>
+    <hardwareInterface>hardware_interface/PositionJointInterface</hardwareInterface>
+    <mechanicalReduction>5</mechanicalReduction>
+    </actuator>
+  </transmission> -->
   <transmission name="tran2">
     <type>transmission_interface/SimpleTransmission</type>
     <joint name="FR_theta2">
-      <hardwareInterface>hardware_interface/JointCommandInterface</hardwareInterface>
+      <hardwareInterface>hardware_interface/PositionJointInterface</hardwareInterface>
     </joint>
     <actuator name="motor2">
-    <hardwareInterface>hardware_interface/JointCommandInterface</hardwareInterface>
+    <hardwareInterface>hardware_interface/PositionJointInterface</hardwareInterface>
     <mechanicalReduction>5</mechanicalReduction>
     </actuator>
@@ -962,8 +913,8 @@
     <type>transmission_interface/SimpleTransmission</type>
     <joint name="FR_theta3">
-      <hardwareInterface>hardware_interface/JointCommandInterface</hardwareInterface>
+      <hardwareInterface>hardware_interface/PositionJointInterface</hardwareInterface>
     </joint>
     <actuator name="motor3">
-    <hardwareInterface>hardware_interface/JointCommandInterface</hardwareInterface>
+    <hardwareInterface>hardware_interface/PositionJointInterface</hardwareInterface>
     <mechanicalReduction>5</mechanicalReduction>
     </actuator>
@@ -972,8 +923,8 @@
     <type>transmission_interface/SimpleTransmission</type>
     <joint name="FL_theta1">
-      <hardwareInterface>hardware_interface/JointCommandInterface</hardwareInterface>
+      <hardwareInterface>hardware_interface/PositionJointInterface</hardwareInterface>
     </joint>
     <actuator name="motor4">
-    <hardwareInterface>hardware_interface/JointCommandInterface</hardwareInterface>
+    <hardwareInterface>hardware_interface/PositionJointInterface</hardwareInterface>
     <mechanicalReduction>5</mechanicalReduction>
     </actuator>
@@ -982,8 +933,8 @@
     <type>transmission_interface/SimpleTransmission</type>
     <joint name="FL_theta2">
-      <hardwareInterface>hardware_interface/JointCommandInterface</hardwareInterface>
+      <hardwareInterface>hardware_interface/PositionJointInterface</hardwareInterface>
     </joint>
     <actuator name="motor5">
-    <hardwareInterface>hardware_interface/JointCommandInterface</hardwareInterface>
+    <hardwareInterface>hardware_interface/PositionJointInterface</hardwareInterface>
     <mechanicalReduction>5</mechanicalReduction>
     </actuator>
@@ -992,8 +943,8 @@
     <type>transmission_interface/SimpleTransmission</type>
     <joint name="FL_theta3">
-      <hardwareInterface>hardware_interface/JointCommandInterface</hardwareInterface>
+      <hardwareInterface>hardware_interface/PositionJointInterface</hardwareInterface>
     </joint>
     <actuator name="motor6">
-    <hardwareInterface>hardware_interface/JointCommandInterface</hardwareInterface>
+    <hardwareInterface>hardware_interface/PositionJointInterface</hardwareInterface>
     <mechanicalReduction>5</mechanicalReduction>
     </actuator>
@@ -1002,8 +953,8 @@
     <type>transmission_interface/SimpleTransmission</type>
     <joint name="RR_theta1">
-      <hardwareInterface>hardware_interface/JointCommandInterface</hardwareInterface>
+      <hardwareInterface>hardware_interface/PositionJointInterface</hardwareInterface>
     </joint>
     <actuator name="motor7">
-    <hardwareInterface>hardware_interface/JointCommandInterface</hardwareInterface>
+    <hardwareInterface>hardware_interface/PositionJointInterface</hardwareInterface>
     <mechanicalReduction>5</mechanicalReduction>
     </actuator>
@@ -1012,8 +963,8 @@
     <type>transmission_interface/SimpleTransmission</type>
     <joint name="RR_theta2">
-      <hardwareInterface>hardware_interface/JointCommandInterface</hardwareInterface>
+      <hardwareInterface>hardware_interface/PositionJointInterface</hardwareInterface>
     </joint>
     <actuator name="motor8">
-    <hardwareInterface>hardware_interface/JointCommandInterface</hardwareInterface>
+    <hardwareInterface>hardware_interface/PositionJointInterface</hardwareInterface>
     <mechanicalReduction>5</mechanicalReduction>
     </actuator>
@@ -1022,8 +973,8 @@
     <type>transmission_interface/SimpleTransmission</type>
     <joint name="RR_theta3">
-      <hardwareInterface>hardware_interface/JointCommandInterface</hardwareInterface>
+      <hardwareInterface>hardware_interface/PositionJointInterface</hardwareInterface>
     </joint>
     <actuator name="motor9">
-    <hardwareInterface>hardware_interface/JointCommandInterface</hardwareInterface>
+    <hardwareInterface>hardware_interface/PositionJointInterface</hardwareInterface>
     <mechanicalReduction>5</mechanicalReduction>
     </actuator>
@@ -1032,8 +983,8 @@
     <type>transmission_interface/SimpleTransmission</type>
     <joint name="RL_theta1">
-      <hardwareInterface>hardware_interface/JointCommandInterface</hardwareInterface>
+      <hardwareInterface>hardware_interface/PositionJointInterface</hardwareInterface>
     </joint>
     <actuator name="motor10">
-    <hardwareInterface>hardware_interface/JointCommandInterface</hardwareInterface>
+    <hardwareInterface>hardware_interface/PositionJointInterface</hardwareInterface>
     <mechanicalReduction>5</mechanicalReduction>
     </actuator>
@@ -1042,8 +993,8 @@
     <type>transmission_interface/SimpleTransmission</type>
     <joint name="RL_theta2">
-      <hardwareInterface>hardware_interface/JointCommandInterface</hardwareInterface>
+      <hardwareInterface>hardware_interface/PositionJointInterface</hardwareInterface>
     </joint>
     <actuator name="motor11">
-    <hardwareInterface>hardware_interface/JointCommandInterface</hardwareInterface>
+    <hardwareInterface>hardware_interface/PositionJointInterface</hardwareInterface>
     <mechanicalReduction>5</mechanicalReduction>
     </actuator>
@@ -1052,8 +1003,8 @@
     <type>transmission_interface/SimpleTransmission</type>
     <joint name="RL_theta3">
-      <hardwareInterface>hardware_interface/JointCommandInterface</hardwareInterface>
+      <hardwareInterface>hardware_interface/PositionJointInterface</hardwareInterface>
     </joint>
     <actuator name="motor12">
-    <hardwareInterface>hardware_interface/JointCommandInterface</hardwareInterface>
+    <hardwareInterface>hardware_interface/PositionJointInterface</hardwareInterface>
     <mechanicalReduction>5</mechanicalReduction>
     </actuator>

File: src/magbot_gazebo/description/urdf/dingo_ros2_control.xacro (robot description, xacro)
@@ -12,4 +12,5 @@
         <state_interface name="velocity"/>
         <state_interface name="effort"/>
+        <param name="initial_position">0.0</param>
       </joint>
       <joint name="FL_theta2">
@@ -18,4 +19,5 @@
         <state_interface name="velocity"/>
         <state_interface name="effort"/>
+        <param name="initial_position">0.0</param>
       </joint>
       <joint name="FL_theta3">
@@ -24,4 +26,5 @@
         <state_interface name="velocity"/>
         <state_interface name="effort"/>
+        <param name="initial_position">0.0</param>
       </joint>
       <!-- FR Joint Group -->
@@ -31,4 +34,5 @@
         <state_interface name="velocity"/>
         <state_interface name="effort"/>
+        <param name="initial_position">0.0</param>
       </joint>
       <joint name="FR_theta2">
@@ -37,4 +41,5 @@
         <state_interface name="velocity"/>
         <state_interface name="effort"/>
+        <param name="initial_position">0.0</param>
       </joint>
       <joint name="FR_theta3">
@@ -43,4 +48,5 @@
         <state_interface name="velocity"/>
         <state_interface name="effort"/>
+        <param name="initial_position">0.0</param>
       </joint>
       <!-- RR Joint Group -->
@@ -50,4 +56,5 @@
         <state_interface name="velocity"/>
         <state_interface name="effort"/>
+        <param name="initial_position">0.0</param>
       </joint>
       <joint name="RR_theta2">
@@ -56,4 +63,5 @@
         <state_interface name="velocity"/>
         <state_interface name="effort"/>
+        <param name="initial_position">0.0</param>
       </joint>
       <joint name="RR_theta3">
@@ -62,4 +70,5 @@
         <state_interface name="velocity"/>
         <state_interface name="effort"/>
+        <param name="initial_position">0.0</param>
       </joint>
       <!-- RL Joint Group -->
@@ -69,4 +78,5 @@
         <state_interface name="velocity"/>
         <state_interface name="effort"/>
+        <param name="initial_position">0.0</param>
       </joint>
       <joint name="RL_theta2">
@@ -75,4 +85,5 @@
         <state_interface name="velocity"/>
         <state_interface name="effort"/>
+        <param name="initial_position">0.0</param>
       </joint>
       <joint name="RL_theta3">
@@ -81,5 +92,115 @@
         <state_interface name="velocity"/>
         <state_interface name="effort"/>
-      </joint>
+        <param name="initial_position">0.0</param>
+      </joint>
+      <!-- Transmissions -->
+      <transmission name="tran1">
+        <plugin>transmission_interface/SimpleTransmission</plugin>
+        <actuator name="motor1" role="actuator1">
+          <mechanical_reduction>5</mechanical_reduction>
+        </actuator>
+        <joint name="FR_theta1" role="joint1">
+          <offset>0.0</offset>
+        </joint>
+      </transmission>
+      <transmission name="tran2">
+        <plugin>transmission_interface/SimpleTransmission</plugin>
+        <actuator name="motor2" role="actuator1">
+          <mechanical_reduction>5</mechanical_reduction>
+        </actuator>
+        <joint name="FR_theta2" role="joint1">
+          <offset>0.0</offset>
+        </joint>
+      </transmission>
+      <transmission name="tran3">
+        <plugin>transmission_interface/SimpleTransmission</plugin>
+        <actuator name="motor3" role="actuator1">
+          <mechanical_reduction>5</mechanical_reduction>
+        </actuator>
+        <joint name="FR_theta3" role="joint1">
+          <offset>0.0</offset>
+        </joint>
+      </transmission>
+      <transmission name="tran4">
+        <plugin>transmission_interface/SimpleTransmission</plugin>
+        <actuator name="motor4" role="actuator1">
+          <mechanical_reduction>5</mechanical_reduction>
+        </actuator>
+        <joint name="FL_theta1" role="joint1">
+          <offset>0.0</offset>
+        </joint>
+      </transmission>
+      <transmission name="tran5">
+        <plugin>transmission_interface/SimpleTransmission</plugin>
+        <actuator name="motor5" role="actuator1">
+          <mechanical_reduction>5</mechanical_reduction>
+        </actuator>
+        <joint name="FL_theta2" role="joint1">
+          <offset>0.0</offset>
+        </joint>
+      </transmission>
+      <transmission name="tran6">
+        <plugin>transmission_interface/SimpleTransmission</plugin>
+        <actuator name="motor6" role="actuator1">
+          <mechanical_reduction>5</mechanical_reduction>
+        </actuator>
+        <joint name="FL_theta3" role="joint1">
+          <offset>0.0</offset>
+        </joint>
+      </transmission>
+      <transmission name="tran7">
+        <plugin>transmission_interface/SimpleTransmission</plugin>
+        <actuator name="motor7" role="actuator1">
+          <mechanical_reduction>5</mechanical_reduction>
+        </actuator>
+        <joint name="RR_theta1" role="joint1">
+          <offset>0.0</offset>
+        </joint>
+      </transmission>
+      <transmission name="tran8">
+        <plugin>transmission_interface/SimpleTransmission</plugin>
+        <actuator name="motor8" role="actuator1">
+          <mechanical_reduction>5</mechanical_reduction>
+        </actuator>
+        <joint name="RR_theta2" role="joint1">
+          <offset>0.0</offset>
+        </joint>
+      </transmission>
+      <transmission name="tran9">
+        <plugin>transmission_interface/SimpleTransmission</plugin>
+        <actuator name="motor9" role="actuator1">
+          <mechanical_reduction>5</mechanical_reduction>
+        </actuator>
+        <joint name="RR_theta3" role="joint1">
+          <offset>0.0</offset>
+        </joint>
+      </transmission>
+      <transmission name="tran10">
+        <plugin>transmission_interface/SimpleTransmission</plugin>
+        <actuator name="motor10" role="actuator1">
+          <mechanical_reduction>5</mechanical_reduction>
+        </actuator>
+        <joint name="RL_theta1" role="joint1">
+          <offset>0.0</offset>
+        </joint>
+      </transmission>
+      <transmission name="tran11">
+        <plugin>transmission_interface/SimpleTransmission</plugin>
+        <actuator name="motor11" role="actuator1">
+          <mechanical_reduction>5</mechanical_reduction>
+        </actuator>
+        <joint name="RL_theta2" role="joint1">
+          <offset>0.0</offset>
+        </joint>
+      </transmission>
+      <transmission name="tran12">
+        <plugin>transmission_interface/SimpleTransmission</plugin>
+        <actuator name="motor12" role="actuator1">
+          <mechanical_reduction>5</mechanical_reduction>
+        </actuator>
+        <joint name="RL_theta3" role="joint1">
+          <offset>0.0</offset>
+        </joint>
+      </transmission>
     </ros2_control>
   </xacro:macro>
