Commit message: Bug in ros2 control

File: src/magbot_gazebo/description/urdf/dingo.urdf.xacro (robot description, xacro)
@@ -613,5 +613,5 @@
       effort="${effort_limit}"
       velocity="3" />
-    <dynamics damping="1000.0" friction="1000.0" />
+    <joint_properties damping="1000.0" friction="1000.0" />
   </joint>
   <joint
@@ -632,5 +632,5 @@
       effort="${effort_limit}"
       velocity="3" />
-    <dynamics damping="1000.0" friction="1000.0" />
+    <joint_properties damping="1000.0" friction="1000.0" />
   </joint>
   <joint
@@ -651,5 +651,5 @@
       effort="${effort_limit}"
       velocity="3" />
-    <dynamics damping="1000.0" friction="1000.0" />
+    <joint_properties damping="1000.0" friction="1000.0" />
   </joint>
   <joint
@@ -683,5 +683,5 @@
       effort="${effort_limit}"
       velocity="3" />
-    <dynamics damping="1000.0" friction="1000.0" />
+    <joint_properties damping="1000.0" friction="1000.0" />
   </joint>
   <joint
@@ -702,5 +702,5 @@
       effort="${effort_limit}"
       velocity="3" />
-    <dynamics damping="1000.0" friction="1000.0" />
+    <joint_properties damping="1000.0" friction="1000.0" />
   </joint>
   <joint
@@ -721,5 +721,5 @@
       effort="${effort_limit}"
       velocity="3" />
-    <dynamics damping="1000.0" friction="1000.0" />
+    <joint_properties damping="1000.0" friction="1000.0" />
   </joint>
   <joint
@@ -753,5 +753,5 @@
       effort="${effort_limit}"
       velocity="3" />
-    <dynamics damping="1000.0" friction="1000.0" />
+    <joint_properties damping="1000.0" friction="1000.0" />
   </joint>
   <joint
@@ -772,5 +772,5 @@
       effort="${effort_limit}"
       velocity="3" />
-    <dynamics damping="1000.0" friction="1000.0" />
+    <joint_properties damping="1000.0" friction="1000.0" />
   </joint>
   <joint
@@ -791,5 +791,5 @@
       effort="${effort_limit}"
       velocity="3" />
-    <dynamics damping="1000.0" friction="1000.0" />
+    <joint_properties damping="1000.0" friction="1000.0" />
   </joint>
   <joint
@@ -823,5 +823,5 @@
       effort="${effort_limit}"
       velocity="3" />
-    <dynamics damping="1000.0" friction="1000.0" />
+    <joint_properties damping="1000.0" friction="1000.0" />
   </joint>
   <joint
@@ -842,5 +842,5 @@
       effort="${effort_limit}"
       velocity="3" />
-    <dynamics damping="1000.0" friction="1000.0" />
+    <joint_properties damping="1000.0" friction="1000.0" />
   </joint>
   <joint
@@ -861,5 +861,5 @@
       effort="${effort_limit}"
       velocity="3" />
-    <dynamics damping="1000.0" friction="1000.0" />
+    <joint_properties damping="1000.0" friction="1000.0" />
   </joint>
   <joint
@@ -880,5 +880,5 @@
     <plugin name="gazebo_ros2_control" filename="libgazebo_ros2_control.so">
       <parameters>$(find magbot_gazebo)/config/dingo_controllers.yaml</parameters>
-      <!-- <ros>
+       <!-- <ros>
        <namespace>/dingo_controller</namespace>
      </ros> -->
@@ -886,5 +886,5 @@
   </gazebo>
   <!-- IMU sensor -->
-  <!-- <gazebo reference="base_link">
+  <gazebo reference="base_link">
     <gravity>true</gravity>
     <sensor name="imu_sensor" type="imu">
@@ -898,5 +898,5 @@
             <type>gaussian</type>
             <mean>0.0</mean>
-            <stddev>0.01</stddev>
+            <stddev>0.01</stddev> <!-- Adjust stddev as needed -->
           </noise>
         </angular_velocity>
@@ -905,5 +905,5 @@
             <type>gaussian</type>
             <mean>0.0</mean>
-            <stddev>0.1</stddev>
+            <stddev>0.1</stddev> <!-- Adjust stddev as needed -->
           </noise>
         </linear_acceleration>
@@ -923,5 +923,5 @@
       </plugin>
     </sensor>
-  </gazebo> -->
+  </gazebo>
   <!-- Joint state publisher plugin -->
   <gazebo>

File: src/magbot_gazebo/description/urdf/dingo_ros2_control.xacro (robot description, xacro)
@@ -12,5 +12,5 @@
         <state_interface name="velocity"/>
         <state_interface name="effort"/>
-        <param name="initial_position">0.0</param>
+        <!-- <param name="initial_position">0.0</param> -->
       </joint>
       <joint name="FL_theta2">
@@ -19,5 +19,5 @@
         <state_interface name="velocity"/>
         <state_interface name="effort"/>
-        <param name="initial_position">0.0</param>
+        <!-- <param name="initial_position">0.0</param> -->
       </joint>
       <joint name="FL_theta3">
@@ -26,5 +26,5 @@
         <state_interface name="velocity"/>
         <state_interface name="effort"/>
-        <param name="initial_position">0.0</param>
+        <!-- <param name="initial_position">0.0</param> -->
       </joint>
       <!-- FR Joint Group -->
@@ -34,5 +34,5 @@
         <state_interface name="velocity"/>
         <state_interface name="effort"/>
-        <param name="initial_position">0.0</param>
+        <!-- <param name="initial_position">0.0</param> -->
       </joint>
       <joint name="FR_theta2">
@@ -41,5 +41,5 @@
         <state_interface name="velocity"/>
         <state_interface name="effort"/>
-        <param name="initial_position">0.0</param>
+        <!-- <param name="initial_position">0.0</param> -->
       </joint>
       <joint name="FR_theta3">
@@ -48,5 +48,5 @@
         <state_interface name="velocity"/>
         <state_interface name="effort"/>
-        <param name="initial_position">0.0</param>
+        <!-- <param name="initial_position">0.0</param> -->
       </joint>
       <!-- RR Joint Group -->
@@ -56,5 +56,5 @@
         <state_interface name="velocity"/>
         <state_interface name="effort"/>
-        <param name="initial_position">0.0</param>
+        <!-- <param name="initial_position">0.0</param> -->
       </joint>
       <joint name="RR_theta2">
@@ -63,5 +63,5 @@
         <state_interface name="velocity"/>
         <state_interface name="effort"/>
-        <param name="initial_position">0.0</param>
+        <!-- <param name="initial_position">0.0</param> -->
       </joint>
       <joint name="RR_theta3">
@@ -70,5 +70,5 @@
         <state_interface name="velocity"/>
         <state_interface name="effort"/>
-        <param name="initial_position">0.0</param>
+        <!-- <param name="initial_position">0.0</param> -->
       </joint>
       <!-- RL Joint Group -->
@@ -78,5 +78,5 @@
         <state_interface name="velocity"/>
         <state_interface name="effort"/>
-        <param name="initial_position">0.0</param>
+        <!-- <param name="initial_position">0.0</param> -->
       </joint>
       <joint name="RL_theta2">
@@ -85,5 +85,5 @@
         <state_interface name="velocity"/>
         <state_interface name="effort"/>
-        <param name="initial_position">0.0</param>
+        <!-- <param name="initial_position">0.0</param> -->
       </joint>
       <joint name="RL_theta3">
@@ -92,115 +92,6 @@
         <state_interface name="velocity"/>
         <state_interface name="effort"/>
-        <param name="initial_position">0.0</param>
+        <!-- <param name="initial_position">0.0</param> -->
       </joint>
-      <!-- Transmissions -->
-      <transmission name="tran1">
-        <plugin>transmission_interface/SimpleTransmission</plugin>
-        <actuator name="motor1" role="actuator1">
-          <mechanical_reduction>5</mechanical_reduction>
-        </actuator>
-        <joint name="FR_theta1" role="joint1">
-          <offset>0.0</offset>
-        </joint>
-      </transmission>
-      <transmission name="tran2">
-        <plugin>transmission_interface/SimpleTransmission</plugin>
-        <actuator name="motor2" role="actuator1">
-          <mechanical_reduction>5</mechanical_reduction>
-        </actuator>
-        <joint name="FR_theta2" role="joint1">
-          <offset>0.0</offset>
-        </joint>
-      </transmission>
-      <transmission name="tran3">
-        <plugin>transmission_interface/SimpleTransmission</plugin>
-        <actuator name="motor3" role="actuator1">
-          <mechanical_reduction>5</mechanical_reduction>
-        </actuator>
-        <joint name="FR_theta3" role="joint1">
-          <offset>0.0</offset>
-        </joint>
-      </transmission>
-      <transmission name="tran4">
-        <plugin>transmission_interface/SimpleTransmission</plugin>
-        <actuator name="motor4" role="actuator1">
-          <mechanical_reduction>5</mechanical_reduction>
-        </actuator>
-        <joint name="FL_theta1" role="joint1">
-          <offset>0.0</offset>
-        </joint>
-      </transmission>
-      <transmission name="tran5">
-        <plugin>transmission_interface/SimpleTransmission</plugin>
-        <actuator name="motor5" role="actuator1">
-          <mechanical_reduction>5</mechanical_reduction>
-        </actuator>
-        <joint name="FL_theta2" role="joint1">
-          <offset>0.0</offset>
-        </joint>
-      </transmission>
-      <transmission name="tran6">
-        <plugin>transmission_interface/SimpleTransmission</plugin>
-        <actuator name="motor6" role="actuator1">
-          <mechanical_reduction>5</mechanical_reduction>
-        </actuator>
-        <joint name="FL_theta3" role="joint1">
-          <offset>0.0</offset>
-        </joint>
-      </transmission>
-      <transmission name="tran7">
-        <plugin>transmission_interface/SimpleTransmission</plugin>
-        <actuator name="motor7" role="actuator1">
-          <mechanical_reduction>5</mechanical_reduction>
-        </actuator>
-        <joint name="RR_theta1" role="joint1">
-          <offset>0.0</offset>
-        </joint>
-      </transmission>
-      <transmission name="tran8">
-        <plugin>transmission_interface/SimpleTransmission</plugin>
-        <actuator name="motor8" role="actuator1">
-          <mechanical_reduction>5</mechanical_reduction>
-        </actuator>
-        <joint name="RR_theta2" role="joint1">
-          <offset>0.0</offset>
-        </joint>
-      </transmission>
-      <transmission name="tran9">
-        <plugin>transmission_interface/SimpleTransmission</plugin>
-        <actuator name="motor9" role="actuator1">
-          <mechanical_reduction>5</mechanical_reduction>
-        </actuator>
-        <joint name="RR_theta3" role="joint1">
-          <offset>0.0</offset>
-        </joint>
-      </transmission>
-      <transmission name="tran10">
-        <plugin>transmission_interface/SimpleTransmission</plugin>
-        <actuator name="motor10" role="actuator1">
-          <mechanical_reduction>5</mechanical_reduction>
-        </actuator>
-        <joint name="RL_theta1" role="joint1">
-          <offset>0.0</offset>
-        </joint>
-      </transmission>
-      <transmission name="tran11">
-        <plugin>transmission_interface/SimpleTransmission</plugin>
-        <actuator name="motor11" role="actuator1">
-          <mechanical_reduction>5</mechanical_reduction>
-        </actuator>
-        <joint name="RL_theta2" role="joint1">
-          <offset>0.0</offset>
-        </joint>
-      </transmission>
-      <transmission name="tran12">
-        <plugin>transmission_interface/SimpleTransmission</plugin>
-        <actuator name="motor12" role="actuator1">
-          <mechanical_reduction>5</mechanical_reduction>
-        </actuator>
-        <joint name="RL_theta3" role="joint1">
-          <offset>0.0</offset>
-        </joint>
-      </transmission>
     </ros2_control>
   </xacro:macro>

Commit message: Robot spawns smoothly + TODO: Correct the driver

File: src/magbot_gazebo/description/urdf/dingo.urdf.xacro (robot description, xacro)
@@ -612,5 +612,5 @@
       effort="${effort_limit}"
       velocity="3" />
-    <joint_properties damping="1000.0" friction="1000.0" />
+    <dynamics damping="0.1" friction="0.1" />
   </joint>
   <joint
@@ -631,5 +631,5 @@
       effort="${effort_limit}"
       velocity="3" />
-    <joint_properties damping="1000.0" friction="1000.0" />
+    <dynamics damping="0.1" friction="0.1" />
   </joint>
   <joint
@@ -650,5 +650,5 @@
       effort="${effort_limit}"
       velocity="3" />
-    <joint_properties damping="1000.0" friction="1000.0" />
+    <dynamics damping="0.1" friction="0.1" />
   </joint>
   <joint
@@ -682,5 +682,5 @@
       effort="${effort_limit}"
       velocity="3" />
-    <joint_properties damping="1000.0" friction="1000.0" />
+    <dynamics damping="0.1" friction="0.1" />
   </joint>
   <joint
@@ -701,5 +701,5 @@
       effort="${effort_limit}"
       velocity="3" />
-    <joint_properties damping="1000.0" friction="1000.0" />
+    <dynamics damping="0.1" friction="0.1" />
   </joint>
   <joint
@@ -720,5 +720,5 @@
       effort="${effort_limit}"
       velocity="3" />
-    <joint_properties damping="1000.0" friction="1000.0" />
+    <dynamics damping="0.1" friction="0.1" />
   </joint>
   <joint
@@ -752,5 +752,5 @@
       effort="${effort_limit}"
       velocity="3" />
-    <joint_properties damping="1000.0" friction="1000.0" />
+    <dynamics damping="0.1" friction="0.1" />
   </joint>
   <joint
@@ -771,5 +771,5 @@
       effort="${effort_limit}"
       velocity="3" />
-    <joint_properties damping="1000.0" friction="1000.0" />
+    <dynamics damping="0.1" friction="0.1" />
   </joint>
   <joint
@@ -790,5 +790,5 @@
       effort="${effort_limit}"
       velocity="3" />
-    <joint_properties damping="1000.0" friction="1000.0" />
+    <dynamics damping="0.1" friction="0.1" />
   </joint>
   <joint
@@ -822,5 +822,5 @@
       effort="${effort_limit}"
       velocity="3" />
-    <joint_properties damping="1000.0" friction="1000.0" />
+    <dynamics damping="0.1" friction="0.1" />
   </joint>
   <joint
@@ -841,5 +841,5 @@
       effort="${effort_limit}"
       velocity="3" />
-    <joint_properties damping="1000.0" friction="1000.0" />
+    <dynamics damping="0.1" friction="0.1" />
   </joint>
   <joint
@@ -860,5 +860,5 @@
       effort="${effort_limit}"
       velocity="3" />
-    <joint_properties damping="1000.0" friction="1000.0" />
+    <dynamics damping="0.1" friction="0.1" />
   </joint>
   <joint
@@ -879,8 +879,26 @@
     <plugin name="gazebo_ros2_control" filename="libgazebo_ros2_control.so">
       <parameters>$(find magbot_gazebo)/config/dingo_controllers.yaml</parameters>
-       <!-- <ros>
-       <namespace>/dingo_controller</namespace>
-     </ros> -->
+      <robot_param>robot_description</robot_param>
+      <robot_param_node>robot_state_publisher</robot_param_node>
     </plugin>
+    <physics type="ode">
+      <ode>
+        <solver>
+          <type>quick</type>
+          <iters>50</iters>
+          <sor>1.3</sor>
+        </solver>
+        <constraints>
+          <cfm>0.00001</cfm>
+          <erp>0.2</erp>
+          <contact_max_correcting_vel>100.0</contact_max_correcting_vel>
+          <contact_surface_layer>0.001</contact_surface_layer>
+        </constraints>
+      </ode>
+      <max_contacts>20</max_contacts>
+      <gravity>0 0 -9.81</gravity>
+    </physics>
+    <real_time_update_rate>250</real_time_update_rate>
+    <max_step_size>0.004</max_step_size>
   </gazebo>
   <gazebo>
@@ -926,6 +944,64 @@
     </sensor>
   </gazebo> -->
+  <gazebo reference="base_link">
+    <gravity>true</gravity>
+    <sensor name="imu_sensor" type="imu">
+      <always_on>true</always_on>
+      <update_rate>100</update_rate>
+      <visualize>true</visualize>
+      <imu>
+        <angular_velocity>
+          <x>
+            <noise type="gaussian">
+              <mean>0.0</mean>
+              <stddev>0.01</stddev>
+            </noise>
+          </x>
+          <y>
+            <noise type="gaussian">
+              <mean>0.0</mean>
+              <stddev>0.01</stddev>
+            </noise>
+          </y>
+          <z>
+            <noise type="gaussian">
+              <mean>0.0</mean>
+              <stddev>0.01</stddev>
+            </noise>
+          </z>
+        </angular_velocity>
+        <linear_acceleration>
+          <x>
+            <noise type="gaussian">
+              <mean>0.0</mean>
+              <stddev>0.1</stddev>
+            </noise>
+          </x>
+          <y>
+            <noise type="gaussian">
+              <mean>0.0</mean>
+              <stddev>0.1</stddev>
+            </noise>
+          </y>
+          <z>
+            <noise type="gaussian">
+              <mean>0.0</mean>
+              <stddev>0.1</stddev>
+            </noise>
+          </z>
+        </linear_acceleration>
+      </imu>
+      <plugin name="imu_plugin" filename="libgazebo_ros_imu_sensor.so">
+        <ros>
+          <namespace>/dingo</namespace>
+          <remapping>~/out:=imu</remapping>
+        </ros>
+        <initial_orientation_as_reference>false</initial_orientation_as_reference>
+        <frame_name>base_link</frame_name>
+      </plugin>
+    </sensor>
+  </gazebo>
   <!-- Joint state publisher plugin -->
-  <gazebo>
+  <!-- <gazebo>
     <plugin name="joint_state_publisher" filename="libgazebo_ros_joint_state_publisher.so">
       <ros>
@@ -947,5 +1023,5 @@
       <joint_name>RL_theta3</joint_name>
     </plugin>
-  </gazebo>
+  </gazebo> -->
   <!-- FR4 friction -->
   <gazebo reference="FR_link4">
@@ -981,3 +1057,10 @@
   </gazebo>
   <xacro:dingo_ros2_control name="DingoRobotSystem" />
+  <gazebo reference="base_link">
+    <selfCollide>true</selfCollide>
+    <mu1>0.2</mu1>
+    <mu2>0.2</mu2>
+    <kp>100000.0</kp>
+    <kd>10.0</kd>
+  </gazebo>
 </robot>

File: src/magbot_gazebo/description/urdf/dingo_ros2_control.xacro (robot description, xacro)
@@ -8,53 +8,77 @@
       <!-- FL Joint Group -->
       <joint name="FL_theta1">
-        <command_interface name="position"/>
-        <state_interface name="position"/>
+        <command_interface name="effort" />
+        <state_interface name="effort" />
+        <state_interface name="position" />
+        <state_interface name="velocity" />
       </joint>
       <joint name="FL_theta2">
-        <command_interface name="position"/>
-        <state_interface name="position"/>
+        <command_interface name="effort" />
+        <state_interface name="effort" />
+        <state_interface name="position" />
+        <state_interface name="velocity" />
       </joint>
       <joint name="FL_theta3">
-        <command_interface name="position"/>
-        <state_interface name="position"/>
+        <command_interface name="effort" />
+        <state_interface name="effort" />
+        <state_interface name="position" />
+        <state_interface name="velocity" />
       </joint>
       <!-- FR Joint Group -->
       <joint name="FR_theta1">
-        <command_interface name="position"/>
-        <state_interface name="position"/>
+        <command_interface name="effort" />
+        <state_interface name="effort" />
+        <state_interface name="position" />
+        <state_interface name="velocity" />
       </joint>
       <joint name="FR_theta2">
-        <command_interface name="position"/>
-        <state_interface name="position"/>
+        <command_interface name="effort" />
+        <state_interface name="effort" />
+        <state_interface name="position" />
+        <state_interface name="velocity" />
       </joint>
       <joint name="FR_theta3">
-        <command_interface name="position"/>
-        <state_interface name="position"/>
+        <command_interface name="effort" />
+        <state_interface name="effort" />
+        <state_interface name="position" />
+        <state_interface name="velocity" />
       </joint>
       <!-- RR Joint Group -->
       <joint name="RR_theta1">
-        <command_interface name="position"/>
-        <state_interface name="position"/>
+        <command_interface name="effort" />
+        <state_interface name="effort" />
+        <state_interface name="position" />
+        <state_interface name="velocity" />
       </joint>
       <joint name="RR_theta2">
-        <command_interface name="position"/>
-        <state_interface name="position"/>
+        <command_interface name="effort" />
+        <state_interface name="effort" />
+        <state_interface name="position" />
+        <state_interface name="velocity" />
       </joint>
       <joint name="RR_theta3">
-        <command_interface name="position"/>
-        <state_interface name="position"/>
+        <command_interface name="effort" />
+        <state_interface name="effort" />
+        <state_interface name="position" />
+        <state_interface name="velocity" />
       </joint>
       <!-- RL Joint Group -->
       <joint name="RL_theta1">
-        <command_interface name="position"/>
-        <state_interface name="position"/>
+        <command_interface name="effort" />
+        <state_interface name="effort" />
+        <state_interface name="position" />
+        <state_interface name="velocity" />
       </joint>
       <joint name="RL_theta2">
-        <command_interface name="position"/>
-        <state_interface name="position"/>
+        <command_interface name="effort" />
+        <state_interface name="effort" />
+        <state_interface name="position" />
+        <state_interface name="velocity" />
       </joint>
       <joint name="RL_theta3">
-        <command_interface name="position"/>
-        <state_interface name="position"/>
+        <command_interface name="effort" />
+        <state_interface name="effort" />
+        <state_interface name="position" />
+        <state_interface name="velocity" />
       </joint>
     </ros2_control>
