Commit message: ROBOT WORKSgit add .

File: src/magbot_gazebo/description/urdf/dingo.urdf.xacro (robot description, xacro)
@@ -892,5 +892,5 @@
         </solver>
         <constraints>
-          <cfm>0.00001</cfm>
+          <cfm>0.0001</cfm>
           <erp>0.2</erp>
           <contact_max_correcting_vel>100.0</contact_max_correcting_vel>
@@ -898,12 +898,9 @@
         </constraints>
       </ode>
-      <max_contacts>20</max_contacts>
+      <max_step_size>0.001</max_step_size>
+      <real_time_factor>1</real_time_factor>
+      <real_time_update_rate>1000</real_time_update_rate>
       <gravity>0 0 -9.81</gravity>
     </physics>
-    <real_time_update_rate>250</real_time_update_rate>
-    <max_step_size>0.004</max_step_size>
-  </gazebo>
-  <gazebo>
-    <real_time_update_rate>50</real_time_update_rate>
   </gazebo>
   <!-- IMU sensor -->

File: src/magbot_gazebo/description/urdf/dingo_ros2_control.xacro (robot description, xacro)
@@ -6,4 +6,23 @@
         <plugin>gazebo_ros2_control/GazeboSystem</plugin>
       </hardware>
+      <!-- FR Joint Group -->
+      <joint name="FR_theta1">
+        <command_interface name="effort" />
+        <state_interface name="effort" />
+        <state_interface name="position" />
+        <state_interface name="velocity" />
+      </joint>
+      <joint name="FR_theta2">
+        <command_interface name="effort" />
+        <state_interface name="effort" />
+        <state_interface name="position" />
+        <state_interface name="velocity" />
+      </joint>
+      <joint name="FR_theta3">
+        <command_interface name="effort" />
+        <state_interface name="effort" />
+        <state_interface name="position" />
+        <state_interface name="velocity" />
+      </joint>
       <!-- FL Joint Group -->
       <joint name="FL_theta1">
@@ -20,23 +39,4 @@
       </joint>
       <joint name="FL_theta3">
-        <command_interface name="effort" />
-        <state_interface name="effort" />
-        <state_interface name="position" />
-        <state_interface name="velocity" />
-      </joint>
-      <!-- FR Joint Group -->
-      <joint name="FR_theta1">
-        <command_interface name="effort" />
-        <state_interface name="effort" />
-        <state_interface name="position" />
-        <state_interface name="velocity" />
-      </joint>
-      <joint name="FR_theta2">
-        <command_interface name="effort" />
-        <state_interface name="effort" />
-        <state_interface name="position" />
-        <state_interface name="velocity" />
-      </joint>
-      <joint name="FR_theta3">
         <command_interface name="effort" />
         <state_interface name="effort" />

Commit message: Refactored Driver code

File: src/magbot_gazebo/description/urdf/dingo.urdf.xacro (robot description, xacro)
@@ -6,18 +6,4 @@
   <link
     name="base_link">
-    <!-- <inertial>
-      <origin xyz="0.0 0.0 0.0"/>
-      <mass value="2.50000000"/>
-      <inertia ixx="0.00664756" ixy="0.00002187" ixz="0.00015428" iyy="0.02996945" iyz="-0.00000064"
-    izz="0.03274274"/>
-    </inertial>-->
-    <!--
-    <inertial>
-      <origin xyz="0.0 0.00126483 -0.00622132"/>
-      <mass value="2.5000000"/>
-      <inertia ixx="0.00664756" ixy="0.00002187" ixz="0.00015428" iyy="0.02996945" iyz="-0.00000064"
-    izz="0.03274274"/>
-    </inertial>
-    -->
     <inertial>
       <origin
@@ -34,12 +20,4 @@
         izz="0.00063853" />
     </inertial>
-    <!--
-    <inertial>
-      <origin xyz="-0.02679290 -0.00012097 0.00457177"/>
-      <mass value="5.0000000"/>
-      <inertia ixx="0.00732760" ixy="-0.00000000" ixz="0.00021940" iyy="0.02995798" iyz="-0.00000002"
-    izz="0.03298004"/>
-    </inertial>
-    -->
     <visual>
       <origin
@@ -904,43 +882,4 @@
     </physics>
   </gazebo>
-  <!-- IMU sensor -->
-  <!-- <gazebo reference="base_link">
-    <gravity>true</gravity>
-    <sensor name="imu_sensor" type="imu">
-      <always_on>true</always_on>
-      <update_rate>100</update_rate>
-      <visualize>true</visualize>
-      <topic>__default_topic__</topic>
-      <imu>
-        <angular_velocity>
-          <noise>
-            <type>gaussian</type>
-            <mean>0.0</mean>
-            <stddev>0.01</stddev>
-          </noise>
-        </angular_velocity>
-        <linear_acceleration>
-          <noise>
-            <type>gaussian</type>
-            <mean>0.0</mean>
-            <stddev>0.1</stddev>
-          </noise>
-        </linear_acceleration>
-      </imu>
-      <pose>0 0 0 0 0 0</pose>
-      <plugin filename="libgazebo_ros_imu_sensor.so" name="imu_plugin">
-        <ros>
-          <namespace>/dingo</namespace>
-          <remapping>~/out:=imu</remapping>
-        </ros>
-        <topicName>imu</topicName>
-        <bodyName>base_link</bodyName>
-        <updateRateHZ>15.0</updateRateHZ>
-        <xyzOffset>0 0 0</xyzOffset>
-        <rpyOffset>0 0 0</rpyOffset>
-        <frameName>base_link</frameName>
-      </plugin>
-    </sensor>
-  </gazebo> -->
   <gazebo reference="base_link">
     <gravity>true</gravity>
@@ -1001,26 +940,4 @@
     </sensor>
   </gazebo>
-  <!-- Joint state publisher plugin -->
-  <gazebo>
-    <plugin name="joint_state_publisher" filename="libgazebo_ros_joint_state_publisher.so">
-      <ros>
-        <namespace>/</namespace>
-        <remapping>~/out:=magbot/joint_states</remapping>
-      </ros>
-      <update_rate>1000</update_rate>
-      <joint_name>FR_theta1</joint_name>
-      <joint_name>FR_theta2</joint_name>
-      <joint_name>FR_theta3</joint_name>
-      <joint_name>FL_theta1</joint_name>
-      <joint_name>FL_theta2</joint_name>
-      <joint_name>FL_theta3</joint_name>
-      <joint_name>RR_theta1</joint_name>
-      <joint_name>RR_theta2</joint_name>
-      <joint_name>RR_theta3</joint_name>
-      <joint_name>RL_theta1</joint_name>
-      <joint_name>RL_theta2</joint_name>
-      <joint_name>RL_theta3</joint_name>
-    </plugin>
-  </gazebo>
   <!-- FR4 friction -->
   <gazebo reference="FR_link4">
