Commit message: Robot spawns in Gazebo

File: src/magbot_gazebo/description/urdf/dingo.urdf (robot description, URDF)
Before this commit: robot dingo, 17 links, 16 joints
Links:
- link FL_link1: geometry collision mesh filename=package://magbot_gazebo/description/meshes/L_link1_collisio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; visual mesh filename=package://magbot_gazebo/description/meshes/FL_link1.dae
- link FL_link2: geometry collision mesh filename=package://magbot_gazebo/description/meshes/L_link2_collisio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; visual mesh filename=package://magbot_gazebo/description/meshes/L_link2.dae
- link FL_link3: geometry collision mesh filename=package://magbot_gazebo/description/meshes/L_link3_collisio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; visual mesh filename=package://magbot_gazebo/description/meshes/L_link3.dae
- link FL_link4: geometry collision mesh filename=package://magbot_gazebo/description/meshes/link4_collision.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; visual mesh filename=package://magbot_gazebo/description/meshes/link4.dae
- link FR_link1: geometry collision mesh filename=package://magbot_gazebo/description/meshes/R_link1_collisio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; visual mesh filename=package://magbot_gazebo/description/meshes/FR_link1.dae
- link FR_link2: geometry collision mesh filename=package://magbot_gazebo/description/meshes/R_link2_collisio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; visual mesh filename=package://magbot_gazebo/description/meshes/R_link2.dae
- link FR_link3: geometry collision mesh filename=package://magbot_gazebo/description/meshes/R_link3_collisio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; visual mesh filename=package://magbot_gazebo/description/meshes/R_link3.dae
- link FR_link4: geometry collision mesh filename=package://magbot_gazebo/description/meshes/link4_collision.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; visual mesh filename=package://magbot_gazebo/description/meshes/link4.dae
- link RL_link1: geometry collision mesh filename=package://magbot_gazebo/description/meshes/L_link1_collisio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; visual mesh filename=package://magbot_gazebo/description/meshes/RL_link1.dae
- link RL_link2: geometry collision mesh filename=package://magbot_gazebo/description/meshes/L_link2_collisio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; visual mesh filename=package://magbot_gazebo/description/meshes/L_link2.dae
- link RL_link3: geometry collision mesh filename=package://magbot_gazebo/description/meshes/L_link3_collisio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; visual mesh filename=package://magbot_gazebo/description/meshes/L_link3.dae
- link RL_link4: geometry collision mesh filename=package://magbot_gazebo/description/meshes/link4_collision.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; visual mesh filename=package://magbot_gazebo/description/meshes/link4.dae
- link RR_link1: geometry collision mesh filename=package://magbot_gazebo/description/meshes/R_link1_collisio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; visual mesh filename=package://magbot_gazebo/description/meshes/RR_link1.dae
- link RR_link2: geometry collision mesh filename=package://magbot_gazebo/description/meshes/R_link2_collisio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; visual mesh filename=package://magbot_gazebo/description/meshes/R_link2.dae
- link RR_link3: geometry collision mesh filename=package://magbot_gazebo/description/meshes/R_link3_collisio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; visual mesh filename=package://magbot_gazebo/description/meshes/R_link3.dae
- link RR_link4: geometry collision mesh filename=package://magbot_gazebo/description/meshes/link4_collision.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; visual mesh filename=package://magbot_gazebo/description/meshes/link4.dae
- link base_link: geometry collision mesh filename=package://magbot_gazebo/description/meshes/base_collision.S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; visual mesh filename=package://magbot_gazebo/description/meshes/base_link.dae

Commit message: Robot spawns and controller loads

File: src/magbot_gazebo/description/urdf/dingo.urdf (robot description, URDF)
Before this commit: robot dingo, 17 links, 16 joints
Links:
- link base_link: mass 0.81776 -> 5.0000000

File: src/magbot_gazebo/description/urdf/dingo.urdf.xacro (robot description, xacro)
@@ -3,8 +3,15 @@
   <!-- Maximum torque -->
   <xacro:property name="effort_limit" value="10" />
+  <!-- The root link can't have inertia so did this -->
+  <!-- <link name="root_dummy_link" />
+  <joint name="root_joint" type="fixed">
+    <parent link="root_dummy_link"/>
+    <child link="base_link"/>
+  </joint> -->
+  <!-- The root link can't have inertia so did this -->
   <!-- base_link -->
   <link
     name="base_link">
-    <inertial>
+    <!-- <inertial>
       <origin
         xyz="0 0 0"
@@ -19,6 +26,5 @@
         iyz="3.2027E-08"
         izz="0.00063853" />
-    </inertial>
-    <!--
+    </inertial> -->
     <inertial>
       <origin xyz="-0.02679290 -0.00012097 0.00457177"/>
@@ -26,5 +32,4 @@
       <inertia ixx="0.00732760" ixy="-0.00000000" ixz="0.00021940" iyy="0.02995798" iyz="-0.00000002" izz="0.03298004"/>
     </inertial>
-    -->
     <visual>
       <origin
@@ -889,127 +894,34 @@
     </plugin>
   </gazebo>
-  <!-- Transmission -->
-  <!-- <transmission name="tran1">
-    <type>transmission_interface/SimpleTransmission</type>
-    <joint name="FR_theta1">
-      <hardwareInterface>hardware_interface/PositionJointInterface</hardwareInterface>
-    </joint>
-    <actuator name="motor1">
-    <hardwareInterface>hardware_interface/PositionJointInterface</hardwareInterface>
-    <mechanicalReduction>5</mechanicalReduction>
-    </actuator>
-  </transmission> -->
-  <transmission name="tran2">
-    <type>transmission_interface/SimpleTransmission</type>
-    <joint name="FR_theta2">
-      <hardwareInterface>hardware_interface/PositionJointInterface</hardwareInterface>
-    </joint>
-    <actuator name="motor2">
-    <hardwareInterface>hardware_interface/PositionJointInterface</hardwareInterface>
-    <mechanicalReduction>5</mechanicalReduction>
-    </actuator>
-  </transmission>
-  <transmission name="tran3">
-    <type>transmission_interface/SimpleTransmission</type>
-    <joint name="FR_theta3">
-      <hardwareInterface>hardware_interface/PositionJointInterface</hardwareInterface>
-    </joint>
-    <actuator name="motor3">
-    <hardwareInterface>hardware_interface/PositionJointInterface</hardwareInterface>
-    <mechanicalReduction>5</mechanicalReduction>
-    </actuator>
-  </transmission>
-  <transmission name="tran4">
-    <type>transmission_interface/SimpleTransmission</type>
-    <joint name="FL_theta1">
-      <hardwareInterface>hardware_interface/PositionJointInterface</hardwareInterface>
-    </joint>
-    <actuator name="motor4">
-    <hardwareInterface>hardware_interface/PositionJointInterface</hardwareInterface>
-    <mechanicalReduction>5</mechanicalReduction>
-    </actuator>
-  </transmission>
-  <transmission name="tran5">
-    <type>transmission_interface/SimpleTransmission</type>
-    <joint name="FL_theta2">
-      <hardwareInterface>hardware_interface/PositionJointInterface</hardwareInterface>
-    </joint>
-    <actuator name="motor5">
-    <hardwareInterface>hardware_interface/PositionJointInterface</hardwareInterface>
-    <mechanicalReduction>5</mechanicalReduction>
-    </actuator>
-  </transmission>
-  <transmission name="tran6">
-    <type>transmission_interface/SimpleTransmission</type>
-    <joint name="FL_theta3">
-      <hardwareInterface>hardware_interface/PositionJointInterface</hardwareInterface>
-    </joint>
-    <actuator name="motor6">
-    <hardwareInterface>hardware_interface/PositionJointInterface</hardwareInterface>
-    <mechanicalReduction>5</mechanicalReduction>
-    </actuator>
-  </transmission>
-  <transmission name="tran7">
-    <type>transmission_interface/SimpleTransmission</type>
-    <joint name="RR_theta1">
-      <hardwareInterface>hardware_interface/PositionJointInterface</hardwareInterface>
-    </joint>
-    <actuator name="motor7">
-    <hardwareInterface>hardware_interface/PositionJointInterface</hardwareInterface>
-    <mechanicalReduction>5</mechanicalReduction>
-    </actuator>
-  </transmission>
-  <transmission name="tran8">
-    <type>transmission_interface/SimpleTransmission</type>
-    <joint name="RR_theta2">
-      <hardwareInterface>hardware_interface/PositionJointInterface</hardwareInterface>
-    </joint>
-    <actuator name="motor8">
-    <hardwareInterface>hardware_interface/PositionJointInterface</hardwareInterface>
-    <mechanicalReduction>5</mechanicalReduction>
-    </actuator>
-  </transmission>
-  <transmission name="tran9">
-    <type>transmission_interface/SimpleTransmission</type>
-    <joint name="RR_theta3">
-      <hardwareInterface>hardware_interface/PositionJointInterface</hardwareInterface>
-    </joint>
-    <actuator name="motor9">
-    <hardwareInterface>hardware_interface/PositionJointInterface</hardwareInterface>
-    <mechanicalReduction>5</mechanicalReduction>
-    </actuator>
-  </transmission>
-  <transmission name="tran10">
-    <type>transmission_interface/SimpleTransmission</type>
-    <joint name="RL_theta1">
-      <hardwareInterface>hardware_interface/PositionJointInterface</hardwareInterface>
-    </joint>
-    <actuator name="motor10">
-    <hardwareInterface>hardware_interface/PositionJointInterface</hardwareInterface>
-    <mechanicalReduction>5</mechanicalReduction>
-    </actuator>
-  </transmission>
-  <transmission name="tran11">
-    <type>transmission_interface/SimpleTransmission</type>
-    <joint name="RL_theta2">
-      <hardwareInterface>hardware_interface/PositionJointInterface</hardwareInterface>
-    </joint>
-    <actuator name="motor11">
-    <hardwareInterface>hardware_interface/PositionJointInterface</hardwareInterface>
-    <mechanicalReduction>5</mechanicalReduction>
-    </actuator>
-  </transmission>
-  <transmission name="tran12">
-    <type>transmission_interface/SimpleTransmission</type>
-    <joint name="RL_theta3">
-      <hardwareInterface>hardware_interface/PositionJointInterface</hardwareInterface>
-    </joint>
-    <actuator name="motor12">
-    <hardwareInterface>hardware_interface/PositionJointInterface</hardwareInterface>
-    <mechanicalReduction>5</mechanicalReduction>
-    </actuator>
-  </transmission>
   <!-- FR4 friction -->
   <gazebo reference="FR_link4">
+    <mu1>1.0</mu1>
+    <mu2>1.0</mu2>
+    <min_depth>0.0002</min_depth> <!-- Updated to min_depth to match Gazebo naming -->
+    <kp>1000000.0</kp>            <!-- Removed value attribute for ROS2 syntax -->
+    <kd>100.0</kd>                <!-- Removed value attribute for ROS2 syntax -->
+  </gazebo>
+  <gazebo reference="FL_link4">
+    <mu1>1.0</mu1>
+    <mu2>1.0</mu2>
+    <min_depth>0.0002</min_depth>
+    <kp>1000000.0</kp>
+    <kd>100.0</kd>
+  </gazebo>
+  <gazebo reference="RR_link4">
+    <mu1>1.0</mu1>
+    <mu2>1.0</mu2>
+    <min_depth>0.0002</min_depth>
+    <kp>1000000.0</kp>
+    <kd>100.0</kd>
+  </gazebo>
+  <gazebo reference="RL_link4">
+    <mu1>1.0</mu1>
+    <mu2>1.0</mu2>
+    <min_depth>0.0002</min_depth>
+    <kp>1000000.0</kp>
+    <kd>100.0</kd>
+  </gazebo>
+  <!-- <gazebo reference="FR_link4">
     <mu1>1.0</mu1>
     <mu2>1.0</mu2>
@@ -1018,5 +930,4 @@
     <kd  value="100.0"/>
   </gazebo>
-  <!-- FL4 friction -->
   <gazebo reference="FL_link4">
     <mu1>1.0</mu1>
@@ -1026,5 +937,4 @@
     <kd  value="100.0"/>
   </gazebo>
-  <!-- RR4 friction -->
   <gazebo reference="RR_link4">
     <mu1>1.0</mu1>
@@ -1034,5 +944,4 @@
     <kd  value="100.0"/>
   </gazebo>
-  <!-- RL4 friction -->
   <gazebo reference="RL_link4">
     <mu1>1.0</mu1>
@@ -1041,5 +950,5 @@
     <kp  value="1000000.0"/>
     <kd  value="100.0"/>
-  </gazebo>
+  </gazebo> -->
   <xacro:dingo_ros2_control name="DingoRobotSystem" />
 </robot>

Commit message: Bug in control

File: src/magbot_gazebo/description/urdf/dingo.urdf (robot description, URDF)
Before this commit: robot dingo, 17 links, 16 joints
Links:
- link base_link: mass 0.81776 -> 2.2

File: src/magbot_gazebo/description/urdf/dingo.urdf.xacro (robot description, xacro)
@@ -1,4 +1,3 @@
 <robot name="dingo" xmlns:xacro="http://www.ros.org/wiki/xacro">
-  <!-- Maximum torque -->
   <xacro:include filename="$(find magbot_gazebo)/description/urdf/dingo_ros2_control.xacro" />
   <!-- Maximum torque -->
@@ -26,5 +25,5 @@
         rpy="0 0 0" />
       <mass
-        value="0.81776" />
+        value="2.2" />
       <inertia
         ixx="0.00058474"
@@ -885,6 +884,9 @@
     </plugin>
   </gazebo>
+  <gazebo>
+    <real_time_update_rate>50</real_time_update_rate>
+  </gazebo>
   <!-- IMU sensor -->
-  <gazebo reference="base_link">
+  <!-- <gazebo reference="base_link">
     <gravity>true</gravity>
     <sensor name="imu_sensor" type="imu">
@@ -898,5 +900,5 @@
             <type>gaussian</type>
             <mean>0.0</mean>
-            <stddev>0.01</stddev> <!-- Adjust stddev as needed -->
+            <stddev>0.01</stddev>
           </noise>
         </angular_velocity>
@@ -905,5 +907,5 @@
             <type>gaussian</type>
             <mean>0.0</mean>
-            <stddev>0.1</stddev> <!-- Adjust stddev as needed -->
+            <stddev>0.1</stddev>
           </noise>
         </linear_acceleration>
@@ -923,5 +925,5 @@
       </plugin>
     </sensor>
-  </gazebo>
+  </gazebo> -->
   <!-- Joint state publisher plugin -->
   <gazebo>
@@ -931,5 +933,5 @@
         <remapping>~/out:=joint_states</remapping>
       </ros>
-      <update_rate>50</update_rate>
+      <update_rate>1000</update_rate>
       <joint_name>FR_theta1</joint_name>
       <joint_name>FR_theta2</joint_name>

File: src/magbot_gazebo/description/urdf/dingo_ros2_control.xacro (robot description, xacro)
@@ -8,77 +8,53 @@
       <!-- FL Joint Group -->
       <joint name="FL_theta1">
-        <command_interface name="effort"/>
+        <command_interface name="position"/>
         <state_interface name="position"/>
-        <state_interface name="velocity"/>
-        <state_interface name="effort"/>
       </joint>
       <joint name="FL_theta2">
-        <command_interface name="effort"/>
+        <command_interface name="position"/>
         <state_interface name="position"/>
-        <state_interface name="velocity"/>
-        <state_interface name="effort"/>
       </joint>
       <joint name="FL_theta3">
-        <command_interface name="effort"/>
+        <command_interface name="position"/>
         <state_interface name="position"/>
-        <state_interface name="velocity"/>
-        <state_interface name="effort"/>
       </joint>
       <!-- FR Joint Group -->
       <joint name="FR_theta1">
-        <command_interface name="effort"/>
+        <command_interface name="position"/>
         <state_interface name="position"/>
-        <state_interface name="velocity"/>
-        <state_interface name="effort"/>
       </joint>
       <joint name="FR_theta2">
-        <command_interface name="effort"/>
+        <command_interface name="position"/>
         <state_interface name="position"/>
-        <state_interface name="velocity"/>
-        <state_interface name="effort"/>
       </joint>
       <joint name="FR_theta3">
-        <command_interface name="effort"/>
+        <command_interface name="position"/>
         <state_interface name="position"/>
-        <state_interface name="velocity"/>
-        <state_interface name="effort"/>
       </joint>
       <!-- RR Joint Group -->
       <joint name="RR_theta1">
-        <command_interface name="effort"/>
+        <command_interface name="position"/>
         <state_interface name="position"/>
-        <state_interface name="velocity"/>
-        <state_interface name="effort"/>
       </joint>
       <joint name="RR_theta2">
-        <command_interface name="effort"/>
+        <command_interface name="position"/>
         <state_interface name="position"/>
-        <state_interface name="velocity"/>
-        <state_interface name="effort"/>
       </joint>
       <joint name="RR_theta3">
-        <command_interface name="effort"/>
+        <command_interface name="position"/>
         <state_interface name="position"/>
-        <state_interface name="velocity"/>
-        <state_interface name="effort"/>
       </joint>
       <!-- RL Joint Group -->
       <joint name="RL_theta1">
-        <command_interface name="effort"/>
+        <command_interface name="position"/>
         <state_interface name="position"/>
-        <state_interface name="velocity"/>
-        <state_interface name="effort"/>
       </joint>
       <joint name="RL_theta2">
-        <command_interface name="effort"/>
+        <command_interface name="position"/>
         <state_interface name="position"/>
-        <state_interface name="velocity"/>
-        <state_interface name="effort"/>
       </joint>
       <joint name="RL_theta3">
-        <command_interface name="effort"/>
+        <command_interface name="position"/>
         <state_interface name="position"/>
-        <state_interface name="velocity"/>
-        <state_interface name="effort"/>
       </joint>
     </ros2_control>

Commit message: Added a simple world

File: src/magbot_gazebo/description/urdf/dingo.urdf (robot description, URDF)
Before this commit: robot dingo, 17 links, 16 joints
Links:
- added link lidar_link, mass 0.1; collision cylinder length=0.05 radius=0.05; visual cylinder length=0.05 radius=0.05
Joints:
- added joint lidar_joint: type fixed, parent base_link, child lidar_link, origin xyz=0 0 0.05 rpy=0 0 0

File: src/magbot_gazebo/description/urdf/dingo.urdf.xacro (robot description, xacro)
@@ -44,4 +44,70 @@
     </collision>
   </link>
+  <!--LIDAR-->
+  <link name="lidar_link">
+    <inertial>
+      <origin xyz="0 0 0" rpy="0 0 0"/>
+      <mass value="0.1"/> <!-- Adjust mass as needed -->
+      <inertia
+        ixx="0.0001" ixy="0.0" ixz="0.0"
+        iyy="0.0001" iyz="0.0"
+        izz="0.0001"/>
+    </inertial>
+    <visual>
+      <origin xyz="0 0 0" rpy="0 0 0"/>
+      <geometry>
+        <cylinder length="0.05" radius="0.05"/> <!-- Adjust dimensions as needed -->
+      </geometry>
+      <material name="blue">
+        <color rgba="0 0 1 1"/> <!-- Blue color for visualization -->
+      </material>
+    </visual>
+    <collision>
+      <origin xyz="0 0 0" rpy="0 0 0"/>
+      <geometry>
+        <cylinder length="0.05" radius="0.05"/> <!-- Adjust dimensions as needed -->
+      </geometry>
+    </collision>
+  </link>
+  <joint name="lidar_joint" type="fixed">
+    <parent link="base_link"/>
+    <child link="lidar_link"/>
+    <origin xyz="0 0 0.05" rpy="0 0 0"/> <!-- Adjust xyz to place the LiDAR on top of the base_link -->
+  </joint>
+  <gazebo reference="lidar_link">
+    <sensor type="ray" name="lidar_sensor">
+      <pose>0 0 0 0 0 0</pose>
+      <visualize>true</visualize>
+      <update_rate>10</update_rate>
+      <ray>
+        <scan>
+          <horizontal>
+            <samples>360</samples>
+            <resolution>1.0</resolution>
+            <min_angle>-3.14159</min_angle> <!-- -180 degrees -->
+            <max_angle>3.14159</max_angle>  <!-- +180 degrees -->
+          </horizontal>
+        </scan>
+        <range>
+          <min>0.1</min>
+          <max>10.0</max>
+          <resolution>0.01</resolution>
+        </range>
+        <noise>
+          <type>gaussian</type>
+          <mean>0.0</mean>
+          <stddev>0.01</stddev>
+        </noise>
+      </ray>
+      <plugin name="gazebo_ros_lidar_controller" filename="libgazebo_ros_ray_sensor.so">
+        <ros>
+          <namespace>/</namespace>
+          <remapping>~/out:=scan</remapping>
+        </ros>
+        <output_type>sensor_msgs/LaserScan</output_type>
+        <frame_name>lidar_link</frame_name>
+      </plugin>
+    </sensor>
+  </gazebo>
   <!-- FL_link1 -->
   <link

Commit message: Did evo tests

File: src/magbot_gazebo/description/urdf/dingo.urdf (robot description, URDF)
Before this commit: robot dingo, 18 links, 17 joints
Links:
- added link base_footprint
Joints:
- added joint base_footprint_joint: type fixed, parent base_link, child base_footprint, origin xyz=0.0 0.0 0.0 rpy=0.0 0.0 0.0

File: src/magbot_gazebo/description/urdf/dingo.urdf.xacro (robot description, xacro)
@@ -44,4 +44,11 @@
     </collision>
   </link>
+  <link name="base_footprint">
+  </link>
+  <joint name="base_footprint_joint" type="fixed">
+      <parent link="base_link"/>
+      <child link="base_footprint"/>
+      <origin xyz="0.0 0.0 0.0" rpy="0.0 0.0 0.0"/>
+  </joint>
   <!--LIDAR-->
   <link name="lidar_link">
@@ -925,5 +932,5 @@
       <ros>
         <namespace>/</namespace>
-        <remapping>~/out:=/magbot/joint_states</remapping>
+        <remapping>~/out:=/joint_states</remapping>
       </ros>
     </plugin>
@@ -1006,4 +1013,16 @@
     </sensor>
   </gazebo>
+  <gazebo>
+    <plugin name="libgazebo_ros_p3d" filename="libgazebo_ros_p3d.so">
+      <ros>
+        <namespace>p3d</namespace>
+        <remapping>odom:=ground_truth</remapping>
+      </ros>
+      <frame_name>world</frame_name>
+      <body_name>base_link</body_name>
+      <update_rate>200.0</update_rate>
+      <gaussian_noise>0.01</gaussian_noise>
+    </plugin>
+  </gazebo>
   <!-- FR4 friction -->
   <gazebo reference="FR_link4">
